Commit message: done manual

File: src/my_bot/urdf/robot.urdf.xacro (robot description, xacro)
@@ -2,3 +2,6 @@
 <robot xmlns:xacro="http://www.ros.org/wiki/xacro" name="robot">
     <xacro:include filename="robot_core.xacro" />
+    <xacro:include filename="gazebo_control.xacro" />
+    <xacro:include filename="lidar.xacro" />
+    <xacro:include filename="imu.xacro" />
 </robot>

File: src/my_bot/urdf/robot_core.xacro (robot description, xacro)
@@ -110,5 +110,5 @@
     <!-- ==================== FRONT LEFT SWIVEL CASTER ==================== -->
     <!-- Khop xoay co banh quanh truc Z -->
-    <joint name="fl_caster_swivel_joint" type="continuous">
+    <joint name="fl_caster_swivel_joint" type="fixed">
         <parent link="chassis"/>
         <child link="fl_caster_swivel"/>
@@ -135,5 +135,5 @@
     </link>
     <!-- Khop quay banh xe lan quanh truc Y -->
-    <joint name="fl_caster_wheel_joint" type="continuous">
+    <joint name="fl_caster_wheel_joint" type="fixed">
         <parent link="fl_caster_swivel"/>
         <child link="fl_caster_wheel"/>
@@ -169,5 +169,5 @@
     <!-- ==================== FRONT RIGHT SWIVEL CASTER ==================== -->
     <!-- Khop xoay co banh quanh truc Z -->
-    <joint name="fr_caster_swivel_joint" type="continuous">
+    <joint name="fr_caster_swivel_joint" type="fixed">
         <parent link="chassis"/>
         <child link="fr_caster_swivel"/>
@@ -194,5 +194,5 @@
     </link>
     <!-- Khop quay banh xe lan quanh truc Y -->
-    <joint name="fr_caster_wheel_joint" type="continuous">
+    <joint name="fr_caster_wheel_joint" type="fixed">
         <parent link="fr_caster_swivel"/>
         <child link="fr_caster_wheel"/>
